File: PCB_EAGLE/V01/V01.sch (EAGLE design)
At the start: 29 parts, among them IC1 MC33269ST-5.0T3, IC2 MC33269D-5.0, IC3 ATMEGA2560-16AU, IC4 TPS77033, J1 POWER_JACKPTH_LOCK, Q1 16MHz, Y1 16MHz

Commit message: 10/22/17
Parts:
- added BLUETOOTH, PA, PB, PC, PD, PE, PF, PH, PJ, PK, PL: (no value), pinhead:PINHD-1X8
- added C12, C13, C14, C15: 33uF, adafruit:C-US025-024X044
- added IC5, IC6: 7805TV, linear:7805TV
- added LED1, LED2, LED3: (no value), pinhead:PINHD-1X2
- added PG: (no value), pinhead:PINHD-1X6
- added PROGRAM: (no value), pinhead:PINHD-2X3
- added Q2, Q3, Q4: 200mA/40V, SparkFun-DiscreteSemi:TRANS_NPN-2N3904
- added R10, R11, R12: PHOTOCELLPTH, SparkFun-Sensors:PHOTOCELLPTH
- added R13, R14, R15: 1k, resistor:R-US_0204/2V
- added SERV01, SERV02, SERV03: (no value), pinhead:PINHD-1X3
- R5, R6: value 10K -> 4.7k
Connections:
- net N$1 renamed POWERIN
- removed net SCL: IC3.(SCL/INT0)PD0, MPU.3, R6.1, TMP102.4
- removed net SDA: IC3.(SDA/INT1)PD1, MPU.4, R5.1, TMP102.3
- removed net VIN: C1.1, C2.1, D1.C, IC1.IN, IC2.VI
- new net 5.0V: C15.1, IC6.VO, Q2.C, Q3.C, Q4.C
- new net 5V: C12.1, IC5.VO, SERV01.2, SERV02.2, SERV03.2
- new net ALT: TMP102.5
- new net DFU: BLUETOOTH.8
- new net INT: MPU.8
- new net N$5: LED1.1, Q3.E
- new net N$6: LED2.1, Q4.E
- new net N$7: LED3.1, Q2.E
- new net PA0: IC3.(AD0)PA0, PA.1, Q3.B
- new net PA1: IC3.(AD1)PA1, PA.2, Q4.B
- new net PA2: IC3.(AD2)PA2, PA.3, Q2.B
- new net PA3: IC3.(AD3)PA3, PA.4
- new net PA4: IC3.(AD4)PA4, PA.5
- new net PA5: IC3.(AD5)PA5, PA.6
- new net PA6: IC3.(AD6)PA6, PA.7
- new net PA7: IC3.(AD7)PA7, PA.8
- new net PB0: IC3.(SS/PCINT0)PB0, PB.1
- new net PB1: IC3.(SCK/PCINT1)PB1, PB.2, PROGRAM.3
- new net PB2: IC3.(MOSI/PCINT2)PB2, PB.3, PROGRAM.4
- new net PB3: IC3.(MISO/PCINT3)PB3, PB.4, PROGRAM.1
- new net PB4: IC3.(OC2A/PCINT4)PB4, PB.5
- new net PB5: IC3.(OC1A/PCINT5)PB5, PB.6, SERV01.1
- new net PB6: IC3.(OC1B/PCINT6)PB6, PB.7, SERV02.1
- new net PB7: IC3.(OC0A/OC1C/PCINT7)PB7, PB.8, SERV03.1
- new net PC0: IC3.(A8)PC0, PC.1
- new net PC1: IC3.(A9)PC1, PC.2
- new net PC2: IC3.(A10)PC2, PC.3
- new net PC3: IC3.(A11)PC3, PC.4
- new net PC4: IC3.(A12)PC4, PC.5
- new net PC5: IC3.(A13)PC5, PC.6
- new net PC6: IC3.(A14)PC6, PC.7
- new net PC7: IC3.(A15)PC7, PC.8
- new net PD0: IC3.(SCL/INT0)PD0, MPU.3, PD.1, R6.1, TMP102.4
- new net PD1: IC3.(SDA/INT1)PD1, MPU.4, PD.2, R5.1, TMP102.3
- new net PD2: IC3.(RXD1/INT2)PD2, PD.3
- new net PD3: IC3.(TXD1/INT3)PD3, PD.4
- new net PD4: IC3.(ICP1)PD4, PD.5
- new net PD5: IC3.(XCK1)PD5, PD.6
- new net PD6: IC3.(T1)PD6, PD.7
- new net PD7: IC3.(T0)PD7, PD.8
- new net PE0: BLUETOOTH.3, IC3.(RXD0/PCIN8)PE0, PE.1
- new net PE1: BLUETOOTH.4, IC3.(TXD0)PE1, PE.2
- new net PE2: IC3.(XCK0/AIN0)PE2, PE.3
- new net PE3: IC3.(OC3A/AIN1)PE3, PE.4
- new net PE4: IC3.(OC3B/INT4)PE4, PE.5
- new net PE5: IC3.(OC3C/INT5)PE5, PE.6
- new net PE6: IC3.(T3/INT6)PE6, PE.7
- new net PE7: IC3.(CLKO/ICP3/INT7)PE7, PE.8
- new net PF0: IC3.(ADC0)PF0, PF.1, R10.P$2, R13.2
- new net PF1: IC3.(ADC1)PF1, PF.2, R11.P$2, R14.2
- new net PF2: IC3.(ADC2)PF2, PF.3, R12.P$2, R15.2
- new net PF3: IC3.(ADC3)PF3, PF.4
- new net PF4: IC3.(ADC4/TCK)PF4, PF.5
- new net PF5: IC3.(ADC5/TMS)PF5, PF.6
- new net PF6: IC3.(ADC6/TDO)PF6, PF.7
- new net PF7: IC3.(ADC7/TDI)PF7, PF.8
- new net PG0: IC3.(WR)PG0, PG.1
- new net PG1: IC3.(RD)PG1, PG.2
- new net PG2: IC3.(ALE)PG2, PG.3
- new net PG3: IC3.(TOSC2)PG3, PG.4
- new net PG4: IC3.(TOSC1)PG4, PG.5
- new net PG5: IC3.(OC0B)PG5, PG.6
- new net PH0: IC3.PH0(RXD2), PH.1
- new net PH1: IC3.PH1(TXD2), PH.2
- new net PH2: IC3.PH2(XCK2), PH.3
- new net PH3: IC3.PH3(OC4A), PH.4
- new net PH4: IC3.PH4(OC4B), PH.5
- new net PH5: IC3.PH5(OC4C), PH.6
- new net PH6: IC3.PH6(OC2B), PH.7
- new net PH7: IC3.PH7(T4), PH.8
- new net PJ0: IC3.PJ0(RXD3/PCINT9), PJ.1
- new net PJ1: IC3.PJ1(TXD3/PCINT10), PJ.2
- new net PJ2: IC3.PJ2(XCK3/PCINT11), PJ.3
- new net PJ3: IC3.PJ3(PCINT12), PJ.4
- new net PJ4: IC3.PJ4(PCINT13), PJ.5
- new net PJ5: IC3.PJ5(PCINT14), PJ.6
- new net PJ6: IC3.PJ6(PCINT15), PJ.7
- new net PJ7: IC3.PJ7, PJ.8
- new net PK0: IC3.PK0(ADC8/PCINT16), PK.1
- new net PK1: IC3.PK1(ADC9/PCINT17), PK.2
- new net PK2: IC3.PK2(ADC10/PCINT18), PK.3
- new net PK3: IC3.PK3(ADC11/PCINT19), PK.4
- new net PK4: IC3.PK4(ADC12/PCINT20), PK.5
- new net PK5: IC3.PK5(ADC13/PCINT21), PK.6
- new net PK6: IC3.PK6(ADC14/PCINT22), PK.7
- new net PK7: IC3.PK7(ADC15/PCINT23), PK.8
- new net PL0: IC3.PL0(ICP4), PL.1
- new net PL1: IC3.PL1(ICP5), PL.2
- new net PL2: IC3.PL2(T5), PL.3
- new net PL3: IC3.PL3(OC5A), PL.4
- new net PL4: IC3.PL4(OC5B), PL.5
- new net PL5: IC3.PL5(OC5C), PL.6
- new net PL6: IC3.PL6, PL.7
- new net PL7: IC3.PL7, PL.8
- new net RTS: BLUETOOTH.6
- new net VCC: C1.1, C13.1, C14.1, C2.1, D1.C, IC1.IN, IC2.VI, IC5.VI, IC6.VI
- new net XCL: MPU.6
- new net XDA: MPU.5
- net +5V: now also BLUETOOTH.5, PROGRAM.2, R10.P$1, R11.P$1, R12.P$1
- net GND: now also BLUETOOTH.1, BLUETOOTH.2, BLUETOOTH.7, C12.2, C13.2, C14.2, C15.2, IC5.GND, IC6.GND, LED1.2, LED2.2, LED3.2, PROGRAM.6, R13.1, R14.1, R15.1, SERV01.3, SERV02.3, SERV03.3; no longer MPU.5, MPU.6, MPU.8, TMP102.5
- net RESET: now also PROGRAM.5
Other:
- note added: "(MISO)"
- note added: "(SCK)"
- note added: "ADC"
- note added: "ADD0"
- note added: "BLUETOOTH"
- note added: "CIS"
- note added: "LED'S"
- note added: "LED1"
- note added: "LED2"
- note added: "LED3"
- note added: "MISO"
- note added: "MOD"
- note added: "MOSI"
- note added: "PhotoCell Logic"
- note added: "Programmer"
- note added: "RX0"
- note added: "Regulator for LED'S"
- note added: "Regulator for Servos"
- note added: "SCK"
- note added: "SCL"
- note added: "SDA"
- note added: "Servo's"
- note added: "TX0"
- note added: "pwm"
